File: hardware/perch-dock/owl_pads.kicad_sch (KiCad schematic)
At the start: 0 parts

Commit message: feat(hardware): draw the perch board and owl dock-pad schematics; perch ERC clean
Parts:
- added J2: To J303: GND, VBUS, DET, GND, Connector_JST:JST_SH_SM04B-SRSS-TB_1x04-1MP_P1.00mm_Horizontal, symbol Connector_Generic_MountingPin:Conn_01x04_MountingPin
- added MB1, MB2: Breakaway, owltunes:MouseBite_2.5mm_2x0.6mm, symbol Mechanical:MountingHole
- added PAD1: DET, TestPoint:TestPoint_Pad_D3.0mm, symbol Connector:TestPoint
- added PAD2: GND, TestPoint:TestPoint_Pad_D3.0mm, symbol Connector:TestPoint
- added PAD3: VBUS, TestPoint:TestPoint_Pad_D3.0mm, symbol Connector:TestPoint
Connections:
- new net PAD_DET: J2.3 (Pin_3), PAD1.1
- new net PAD_GND: J2.1 (Pin_1), J2.4 (Pin_4), J2.MP (MountPin), PAD2.1
- new net PAD_VBUS: J2.2 (Pin_2), PAD3.1
