File: hardware/perch-dock/perch.kicad_sch (KiCad schematic)
At the start: 0 parts

Commit message: feat(hardware): draw the perch board and owl dock-pad schematics; perch ERC clean
Parts:
- added C1: 10uF, Capacitor_SMD:C_0603_1608Metric, symbol Device:C
- added C2: 100nF, Capacitor_SMD:C_0402_1005Metric, symbol Device:C
- added D1: SMF5.0A, Diode_SMD:D_SOD-123F, symbol Device:D_Zener
- added D2: LESD5D5.0CT1G, Diode_SMD:D_SOD-523, symbol Device:D_TVS
- added F1: 1.1A hold, Fuse:Fuse_1206_3216Metric, symbol Device:Polyfuse
- added H1, H2: M2, MountingHole:MountingHole_2.2mm_M2, symbol Mechanical:MountingHole
- added J1: USB-C power, Connector_USB:USB_C_Receptacle_HRO_TYPE-C-31-M-12, symbol Connector:USB_C_Receptacle_USB2.0_16P
- added LED1: red, LED_SMD:LED_0603_1608Metric, symbol Device:LED
- added P1: Pogo DET, owltunes:PogoPin_Xinyangze_YZ71215080P-02, symbol Connector_Generic:Conn_01x01
- added P2: Pogo GND, owltunes:PogoPin_Xinyangze_YZ71215080P-02, symbol Connector_Generic:Conn_01x01
- added P3: Pogo VBUS, owltunes:PogoPin_Xinyangze_YZ71215080P-02, symbol Connector_Generic:Conn_01x01
- added R1, R2: 5.1k, Resistor_SMD:R_0402_1005Metric, symbol Device:R
- added R3: 10k, Resistor_SMD:R_0402_1005Metric, symbol Device:R
- added R4: 4.7k, Resistor_SMD:R_0402_1005Metric, symbol Device:R
Connections:
- new net DOCK_ID: D2.1 (A1), P1.1 (Pin_1), R3.1
- new net GND: C1.2, C2.2, D1.2 (A), D2.2 (A2), J1.A1 (GND), J1.A12 (GND), J1.B1 (GND), J1.B12 (GND), J1.SH (SHIELD), LED1.1 (K), P2.1 (Pin_1), R1.2, R2.2, R3.2
- new net LED_A: LED1.2 (A), R4.2
- new net PERCH_CC1: J1.A5 (CC1), R1.1
- new net PERCH_CC2: J1.B5 (CC2), R2.1
- new net VBUS_IN: D1.1 (K), F1.1, J1.A4 (VBUS), J1.A9 (VBUS), J1.B4 (VBUS), J1.B9 (VBUS)
- new net VBUS_OUT: C1.1, C2.1, F1.2, P3.1 (Pin_1), R4.1
- no-connect marks 0 -> 6

Commit message: fix(hardware): move the CPL points of U201, J201 and the perch J1 to JLC's origins
The Fabrication Toolkit puts an SMD part's CPL point on the KiCad footprint's anchor; JLC places
its EasyEDA footprint by that footprint's origin. Fitting every assembled part's EasyEDA
footprint onto the board pads by pad number puts the two within 0.075 mm for all parts but
three, where the KiCad anchor is the body centre and EasyEDA's origin is near the pad pattern's
centre:

- U201 (ESP32-S3-WROOM-1, C2913202), bottom, KiCad rotation 180: EasyEDA origin at owl
  (0, 26.723), anchor (0, 30.35). The toolkit turns a bottom offset (x, y) at 180 into (-x, y),
  so FT Position Offset "0,-3.627". CPL (0, 30.35) -> (0, 26.723).
- J201 (TYPE-C-31-M-12, C165948), bottom, rotation 180: origin (-12, -32.229), anchor
  (-12, -33.8): "0,1.571". CPL (-12, -33.8) -> (-12, -32.229).
- Perch J1 (same receptacle), top, rotation 90: the toolkit turns (x, y) into (-y, x); origin
  (12.229, -1.5), anchor (13.8, -1.5): "0,1.571". CPL (13.8, -1.5) -> (12.229, -1.5).

Stored like the rotation offsets: design.toml position_offset, the symbol field, and the
footprint field through hw_sync.py (FIELDS gains "FT Position Offset"); hw_bom.py checks symbol
against design.toml and the sync test checks footprints against design.toml on both boards.
The review and ordering.md say the preview checks these three positions as well as rotations.

hw_fab 0 errors on both boards (main top 6, bottom 81; perch top 15), ERC 0, DRC 0/0/0 with
parity on both, check_all 0, tools tests 110 passed.
Parts:
- J1: FT Position Offset (none) -> 0,1.571
Changed lines of the file:
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@@
+			)
+		)
+		(property "FT Position Offset" "0,1.571"
+			(at 50.8 78.74 0)
+			(hide yes)
+			(show_name no)
+			(do_not_autoplace no)
+			(effects
+				(font
+					(size 1.27 1.27)
+				)
 			)
 		)
