File: hardware/perch-dock/perch-dock.kicad_pcb (KiCad board)
At the start: 2 copper layers, 34 x 29 mm, 22 parts, among them J1 USB-C power, J2 To J303: GND, VBUS, DET, GND, P1 Pogo DET, P2 Pogo GND, P3 Pogo VBUS

Commit message: feat(tools): draw each board's own silkscreen marks and keep references clear of them
tools/hw/hw_silk.py draws a board's name, owner mark, licence, date,
JLC order-number mark, connector and test pad labels and extra pin 1
marks from data (owl frame, KiCad x - 100, 100 - KiCad y), back side
text mirrored, all in a "hw_silk" KiCad group that a re-run replaces
(Board.Delete, with a fresh-interpreter test). A test checks that every
mark meets JLC's 0.8 mm / 0.15 mm (1.0 mm for "Tyukov Inc"), that both
boards carry the owner mark and that JLCJLCJLCJLC is on the main board's
back.

hw_place.py's reference placement now also keeps clear of every
footprint silkscreen drawing and every board silkscreen item. Before, it
only avoided pads, holes and other references, which left C304 over
U301's outline, R210 over J202's and SW201/SW202 over their own. Two
new tests place a board text and another footprint's outline on R1's
first free spot; both fail on the old code.

Perch board: "Tyukov Inc" on F.Silkscreen, 1.0 mm high, 0.15 mm
stroke, below the pogo pins and clear of the neck (owner request, 11
October). Perch DRC 0; hw_fab.py perch-dock 0 fabrication errors.
The main board's marks are drawn in the silkscreen step after routing.
Other:
- board text added: "Tyukov Inc"
Changed lines of the file:
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@@
+		)
+	)
+	(gr_text "Tyukov Inc"
+		(locked yes)
+		(at 98 106.2 0)
+		(layer "F.SilkS")
+		(effects
+			(font
+				(size 1 1)
+				(thickness 0.15)
+			)
 		)
 	)
@@
 		)
 	)
+	(group "hw_silk"
+		(members "ab3b15dc-9bb4-4aad-a069-49172fffc447")
+	)
 	(embedded_fonts no)

Commit message: fix(hardware): key the dock-pad board so it only fits with J2 towards J303
The dock-pad board and its recess were symmetric, so the board could be glued
in turned round, which puts the perch's 5 V on GPIO1 through the DET pad.
The pad section now has a 3.0 mm round-ended notch in its DET end, and the
back cover's recess a tongue that fills it up to the board's back face:
turned or turned over, the board stands 1.6 mm proud and cannot be glued
flat. The pad section also carries "J2 towards J303 >" on its silkscreen.

assembly.md step 7 states the orientation and a meter check before the first
dock (J303 pin 2 to the pad nearest J2, pin 3 to the farthest); step 8 says
which side "right" means when seen from the back. bringup.md reads DOCK_DET
on the first dock: about 0.33 V is right, 3 V or more means undock at once.
Other:
- outline, holes or cut-outs redrawn
- board text added: "J2 towards J303 >"
Changed lines of the file:
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@@
+	(gr_line
+		(start 86 113)
+		(end 86 115.5)
+		(stroke
+			(width 0.05)
+			(type default)
+		)
+		(layer "Edge.Cuts")
+	)
 	(gr_line
 		(start 86 113)
@@
 	)
 	(gr_line
-		(start 86 121)
-		(end 86 113)
+		(start 86 115.5)
+		(end 87 115.5)
+		(stroke
+			(width 0.05)
+			(type default)
+		)
+		(layer "Edge.Cuts")
+	)
+	(gr_line
+		(start 86 118.5)
+		(end 86 121)
+		(stroke
+			(width 0.05)
+			(type default)
+		)
+		(layer "Edge.Cuts")
+	)
+	(gr_arc
+		(start 87 115.5)
+		(mid 88.5 117)
+		(end 87 118.5)
+		(stroke
+			(width 0.05)
+			(type default)
+		)
+		(layer "Edge.Cuts")
+	)
+	(gr_line
+		(start 87 118.5)
+		(end 86 118.5)
 		(stroke
 			(width 0.05)
@@
 	(gr_text "OWL DOCK PADS"
 		(at 96.5 114.6 0)
+		(layer "F.SilkS")
+		(effects
+			(font
+				(size 0.8 0.8)
+				(thickness 0.15)
+			)
+		)
+	)
+	(gr_text "J2 towards J303 >"
+		(locked yes)
+		(at 97.5 117.6 0)
 		(layer "F.SilkS")
 		(effects
@@
 	)
 	(group "hw_silk"
-		(members "ab3b15dc-9bb4-4aad-a069-49172fffc447")
+		(members "0b384dee-df7d-4538-b4d4-9e23f301cf31" "3ddfdda5-50f7-4882-8a61-c2083303e283")
 	)
 	(embedded_fonts no)
