File: hardware/owl-mainboard/power.kicad_sch (KiCad schematic)
At the start: 0 parts

Commit message: feat(hardware): draw the main board power sheet (charger, gauge, 3.3 V, display switch)
Parts:
- added C101, C103, C105, C111: 10uF, Capacitor_SMD:C_0603_1608Metric, symbol Device:C
- added C102, C107, C108: 22uF, Capacitor_SMD:C_0603_1608Metric, symbol Device:C
- added C104: 1uF, Capacitor_SMD:C_0402_1005Metric, symbol Device:C
- added C106, C109, C112: 100nF, Capacitor_SMD:C_0402_1005Metric, symbol Device:C
- added C110: 1nF, Capacitor_SMD:C_0402_1005Metric, symbol Device:C
- added D101, D102: PMEG2020EH, Diode_SMD:D_SOD-123F, symbol Device:D_Schottky
- added H1, H2, H3, H4: M2 bezel, MountingHole:MountingHole_2.2mm_M2, symbol Mechanical:MountingHole
- added H5, H6, H7, H8: M2 body, MountingHole:MountingHole_2.2mm_M2, symbol Mechanical:MountingHole
- added J101: Battery +, NTC, -, Connector_JST:JST_PH_S3B-PH-SM4-TB_1x03-1MP_P2.00mm_Horizontal, symbol Connector_Generic_MountingPin:Conn_01x03_MountingPin
- added L101: 0.47uH, owltunes:L_Murata_DFE201612E, symbol Device:L
- added R101, R102: 2k, Resistor_SMD:R_0402_1005Metric, symbol Device:R
- added R103, R104, R105, R106, R108, R109: 100k, Resistor_SMD:R_0402_1005Metric, symbol Device:R
- added R107: 560k, Resistor_SMD:R_0402_1005Metric, symbol Device:R
- added TP101: VIN_CHG, TestPoint:TestPoint_Pad_D1.0mm, symbol Connector:TestPoint
- added TP102: VSYS, TestPoint:TestPoint_Pad_D1.0mm, symbol Connector:TestPoint
- added TP103: VBAT, TestPoint:TestPoint_Pad_D1.0mm, symbol Connector:TestPoint
- added TP104: +3V3, TestPoint:TestPoint_Pad_D1.0mm, symbol Connector:TestPoint
- added TP105: DISP_3V3, TestPoint:TestPoint_Pad_D1.0mm, symbol Connector:TestPoint
- added TP106: GND, TestPoint:TestPoint_Pad_D1.0mm, symbol Connector:TestPoint
- added TP107: GAUGE_ALRT, TestPoint:TestPoint_Pad_D1.0mm, symbol Connector:TestPoint
- added U101: BQ24073RGTR, Package_DFN_QFN:VQFN-16-1EP_3x3mm_P0.5mm_EP1.6x1.6mm, symbol Battery_Management:BQ24073RGT
- added U102: MAX17048G+T10, owltunes:Maxim_TDFN-8-1EP_2x2mm_P0.5mm, symbol owltunes:MAX17048G+T10
- added U103: TPS63802DLAR, owltunes:TI_DLA_VSON-10_2x3mm_P0.5mm, symbol owltunes:TPS63802DLAR
- added U104: TPS22917DBVR, Package_TO_SOT_SMD:SOT-23-6, symbol Power_Management:TPS22917DBV
Connections:
- new net +3V3: C107.1, C108.1, C109.1, C110.1, R105.1, R106.1, R107.1, TP104.1, U103.6 (VOUT), U104.1 (VIN)
- new net BAT_NTC: J101.2 (Pin_2), U101.1 (TS)
- new net CHG_EN2: R103.2, U101.5 (EN2)
- new net CHG_ILIM: R102.1, U101.12 (ILIM)
- new net CHG_ISET: R101.1, U101.16 (ISET)
- new net CHG_PGOOD: R105.2, U101.7 (~{PGOOD})
- new net CHG_STAT: R106.2, U101.9 (~{CHG})
- new net CHG_SUSPEND: R104.1, U101.6 (EN1)
- new net DISP_3V3: C111.1, C112.1, TP105.1, U104.5 (QOD), U104.6 (VOUT)
- new net DISP_EN: R109.1, U104.3 (ON)
- new net ESP_EN: U103.5 (PG)
- new net GAUGE_ALRT: TP107.1, U102.5 (~{ALRT})
- new net GND: C101.2, C102.2, C103.2, C104.2, C105.2, C106.2, C107.2, C108.2, C109.2, C111.2, C112.2, J101.3 (Pin_3), J101.MP (MountPin), R101.2, R102.2, R104.2, R108.2, R109.2, TP106.1, U101.15 (TD), U101.17 (VSS), U101.4 (~{CE}), U101.8 (VSS), U102.1 (CTG), U102.4 (GND), U102.6 (QSTRT), U102.9 (EP), U103.2 (MODE), U103.3 (AGND), U103.8 (GND), U104.2 (GND)
- new net I2C_SCL: U102.7 (SCL)
- new net I2C_SDA: U102.8 (SDA)
- new net LS_CT: C110.2, U104.4 (CT)
- new net TPS_FB: R107.2, R108.1, U103.4 (FB)
- new net TPS_L1: L101.1, U103.9 (L1)
- new net TPS_L2: L101.2, U103.7 (L2)
- new net VBAT: C103.1, C104.1, J101.1 (Pin_1), TP103.1, U101.2 (BAT), U101.3 (BAT), U102.2 (CELL), U102.3 (VDD)
- new net VBUS_DOCK: D102.2 (A)
- new net VBUS_USB: D101.2 (A)
- new net VIN_CHG: C101.1, D101.1 (K), D102.1 (K), R103.1, TP101.1, U101.13 (IN)
- new net VSYS: C102.1, C105.1, C106.1, TP102.1, U101.10 (OUT), U101.11 (OUT), U103.1 (EN), U103.10 (VIN)
- no-connect marks 0 -> 1
Other:
- note added: "3.3 V buck-boost (TPS63802), PG releases the ESP32 EN"
- note added: "Charger and power path (BQ24073), battery"
- note added: "Display power switch (TPS22917)"
- note added: "Fuel gauge (MAX17048, I2C 0x36)"
- note added: "H1-H4: bezel screws, H5-H8: body screws, positions from mech/contract.json"
- note added: "Inputs: USB (J201) and dock (J303) ORed by Schottky diodes"
- note added: "Mechanical"

Commit message: fix(hardware): limit the charger input to USB 2.0 default power and keep the USB attach capacitance under 10 uF
Parts:
- C101: value 10uF -> 4.7uF; LCSC Part # C19702 -> C19666; MPN CL10A106KP8NNNC -> CL10A475KO8NNNC
- R102: value 2k -> 3.3k; LCSC Part # C4109 -> C25890; MPN 0402WGF2001TCE -> 0402WGF3301TCE
Changed lines of the file:
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@@
 		)
 	)
-	(text_box "Values and why (datasheets: BQ24073 SLUS810N section 8.5; TPS63802 SLVSEU9D section 10; TPS22917 SLVSDW8B section 6)\n- Inputs: VBUS_USB and VBUS_DOCK each reach VIN_CHG through a PMEG2020EH Schottky (about 0.38 V at 0.8 A),\n  so neither input, nor a shorted dock pad, can back-feed the other or the USB host. TVS diodes sit at the connectors.\n- ISET 2.0k: ICHG = KISET / RISET = 890 / 2000 = 0.445 A (KISET 797 to 975: 0.40 to 0.49 A), 0.45 C for the\n  1000 mAh pack. Precharge 88 / 2000 = 44 mA.\n- ILIM 2.0k: IIN = KILIM / RILIM = 1610 / 2000 = 0.805 A (1500 to 1720: 0.75 to 0.86 A), inside the USB 3 default 900 mA.\n- EN2 100k to VIN_CHG, EN1 from GPIO45 with 100k to GND: (EN2, EN1) = (1, 0) selects the ILIM resistor on any input;\n  GPIO45 high gives (1, 1), USB suspend. The pull-up only draws current while input power is present\n  (EN pins have 285k internal pull-downs).\n- CE and TD to GND (charging enabled, termination on), TMR open (30 min precharge and 5 h fast-charge timers).\n- TS to the pack's 10k NTC on J101 pin 2: 75 uA bias, charging stops below about 0 to 4 C (VCOLD 2.1 V, 28k)\n  and above about 47 to 51 C (VHOT 0.30 V, 4.0k) for an NTC beta of 3950 to 3380.\n- TPS63802: VOUT = 0.5 x (1 + 560k / 100k) = 3.300 V; R2 = 100k is the datasheet maximum; MODE low (power save);\n  EN to VSYS (always on); L = 0.47 uH; 10 uF + 100 nF in, 2 x 22 uF + 100 nF out.\n  PG (open drain) is ESP_EN: 10k to +3V3 and 1 uF on the mcu_usb sheet, so the module leaves reset only in regulation.\n- TPS22917: CT 1 nF from CT to VIN, QOD tied to VOUT (fast discharge when the panel is switched off),\n  ON pulled down by 100k (GPIO46 strap must be low at reset).\n- MAX17048: CELL and VDD to VBAT, CTG and QSTRT to GND, ALRT only to TP107; I2C pull-ups are on the periph sheet."
+	(text_box "Values and why (datasheets: BQ24073 SLUS810N section 8.5; TPS63802 SLVSEU9D section 10; TPS22917 SLVSDW8B section 6)\n- Inputs: VBUS_USB and VBUS_DOCK each reach VIN_CHG through a PMEG2020EH Schottky (under 0.38 V at the input limit),\n  so neither input, nor a shorted dock pad, can back-feed the other or the USB host. TVS diodes sit at the connectors.\n  C101 4.7 uF (IN takes 1 to 10 uF) keeps the capacitance a USB host sees through D101 within USB's 10 uF.\n- ISET 2.0k: ICHG = KISET / RISET = 890 / 2000 = 0.445 A (KISET 797 to 975: 0.40 to 0.49 A), 0.45 C for the\n  1000 mAh pack. Precharge 88 / 2000 = 44 mA.\n- ILIM 3.3k: IIN = KILIM / RILIM = 1525 / 3300 = 0.46 A (KILIM 1330 to 1720 for 200 to 500 mA: 0.40 to 0.52 A),\n  USB 2.0 default power: the board has plain 5.1k Rd and does not read CC, and VIN-DPM is off in ILIM mode.\n  When the system load and ICHG together exceed the limit, the charger cuts ICHG (DPPM). Faster charging needs CC sensing.\n- EN2 100k to VIN_CHG, EN1 from GPIO45 with 100k to GND: (EN2, EN1) = (1, 0) selects the ILIM resistor on any input;\n  GPIO45 high gives (1, 1), USB suspend. The pull-up only draws current while input power is present\n  (EN pins have 285k internal pull-downs).\n- CE and TD to GND (charging enabled, termination on), TMR open (30 min precharge and 5 h fast-charge timers).\n- TS to the pack's 10k NTC on J101 pin 2: 75 uA bias, charging stops below about 0 to 4 C (VCOLD 2.1 V, 28k)\n  and above about 47 to 51 C (VHOT 0.30 V, 4.0k) for an NTC beta of 3950 to 3380.\n- TPS63802: VOUT = 0.5 x (1 + 560k / 100k) = 3.300 V; R2 = 100k is the datasheet maximum; MODE low (power save);\n  EN to VSYS (always on); L = 0.47 uH; 10 uF + 100 nF in, 2 x 22 uF + 100 nF out.\n  PG (open drain) is ESP_EN: 10k to +3V3 and 1 uF on the mcu_usb sheet, so the module leaves reset only in regulation.\n- TPS22917: CT 1 nF from CT to VIN, QOD tied to VOUT (fast discharge when the panel is switched off),\n  ON pulled down by 100k (GPIO46 strap must be low at reset).\n- MAX17048: CELL and VDD to VBAT, CTG and QSTRT to GND, ALRT only to TP107; I2C pull-ups are on the periph sheet."
 		(exclude_from_sim no)
 		(at 20.32 223.52 0)
-		(size 130.81 40.64)
+		(size 130.81 46.99)
 		(margins 1.27 1.27 1.27 1.27)
 		(stroke
@@
 			)
 		)
-		(property "Value" "2k"
+		(property "Value" "3.3k"
 			(at 111.76 118.11 0)
 			(show_name no)
@@
 			)
 		)
-		(property "LCSC Part #" "C4109"
+		(property "LCSC Part #" "C25890"
 			(at 109.22 116.84 0)
 			(hide yes)
@@
 			)
 		)
-		(property "MPN" "0402WGF2001TCE"
+		(property "MPN" "0402WGF3301TCE"
 			(at 109.22 116.84 0)
 			(hide yes)
@@
 			)
 		)
-		(property "Value" "10uF"
+		(property "Value" "4.7uF"
 			(at 77.47 60.96 0)
 			(show_name no)
@@
 			)
 		)
-		(property "LCSC Part #" "C19702"
+		(property "LCSC Part #" "C19666"
 			(at 73.66 59.69 0)
 			(hide yes)
@@
 			)
 		)
-		(property "MPN" "CL10A106KP8NNNC"
+		(property "MPN" "CL10A475KO8NNNC"
 			(at 73.66 59.69 0)
 			(hide yes)

Commit message: feat(hardware): draw the main board MCU, USB-C and button sheet
The mcu_usb sheet carries the ESP32-S3-WROOM-1-N16R8 with 22 uF + 100 nF at
its 3V3 pin, the EN network (10k, 1 uF, reset pad), the GPIO0 pull-up with
the boot pads, the 32.768 kHz crystal with 18 pF load capacitors, USB-C with
a separate 5.1k Rd per CC pin, USBLC6-2SC6, 22 ohm series resistors and the
VBUS TVS, the three buttons with 100k pull-ups and 10 nF, the J202 expansion
connector with 10k pull-ups, the UART pads, a notes box and the GPIO table.

TPS63802 PG now reaches ESP_EN through R212 (1k) on its own net TPS_PG, so
the open-drain PG output no longer discharges the 1 uF EN capacitor directly.
Connections:
- net ESP_EN renamed TPS_PG
Changed lines of the file:
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@@
 		)
 	)
-	(text_box "Values and why (datasheets: BQ24073 SLUS810N section 8.5; TPS63802 SLVSEU9D section 10; TPS22917 SLVSDW8B section 6)\n- Inputs: VBUS_USB and VBUS_DOCK each reach VIN_CHG through a PMEG2020EH Schottky (under 0.38 V at the input limit),\n  so neither input, nor a shorted dock pad, can back-feed the other or the USB host. TVS diodes sit at the connectors.\n  C101 4.7 uF (IN takes 1 to 10 uF) keeps the capacitance a USB host sees through D101 within USB's 10 uF.\n- ISET 2.0k: ICHG = KISET / RISET = 890 / 2000 = 0.445 A (KISET 797 to 975: 0.40 to 0.49 A), 0.45 C for the\n  1000 mAh pack. Precharge 88 / 2000 = 44 mA.\n- ILIM 3.3k: IIN = KILIM / RILIM = 1525 / 3300 = 0.46 A (KILIM 1330 to 1720 for 200 to 500 mA: 0.40 to 0.52 A),\n  USB 2.0 default power: the board has plain 5.1k Rd and does not read CC, and VIN-DPM is off in ILIM mode.\n  When the system load and ICHG together exceed the limit, the charger cuts ICHG (DPPM). Faster charging needs CC sensing.\n- EN2 100k to VIN_CHG, EN1 from GPIO45 with 100k to GND: (EN2, EN1) = (1, 0) selects the ILIM resistor on any input;\n  GPIO45 high gives (1, 1), USB suspend. The pull-up only draws current while input power is present\n  (EN pins have 285k internal pull-downs).\n- CE and TD to GND (charging enabled, termination on), TMR open (30 min precharge and 5 h fast-charge timers).\n- TS to the pack's 10k NTC on J101 pin 2: 75 uA bias, charging stops below about 0 to 4 C (VCOLD 2.1 V, 28k)\n  and above about 47 to 51 C (VHOT 0.30 V, 4.0k) for an NTC beta of 3950 to 3380.\n- TPS63802: VOUT = 0.5 x (1 + 560k / 100k) = 3.300 V; R2 = 100k is the datasheet maximum; MODE low (power save);\n  EN to VSYS (always on); L = 0.47 uH; 10 uF + 100 nF in, 2 x 22 uF + 100 nF out.\n  PG (open drain) is ESP_EN: 10k to +3V3 and 1 uF on the mcu_usb sheet, so the module leaves reset only in regulation.\n- TPS22917: CT 1 nF from CT to VIN, QOD tied to VOUT (fast discharge when the panel is switched off),\n  ON pulled down by 100k (GPIO46 strap must be low at reset).\n- MAX17048: CELL and VDD to VBAT, CTG and QSTRT to GND, ALRT only to TP107; I2C pull-ups are on the periph sheet."
+	(text_box "Values and why (datasheets: BQ24073 SLUS810N section 8.5; TPS63802 SLVSEU9D section 10; TPS22917 SLVSDW8B section 6)\n- Inputs: VBUS_USB and VBUS_DOCK each reach VIN_CHG through a PMEG2020EH Schottky (under 0.38 V at the input limit),\n  so neither input, nor a shorted dock pad, can back-feed the other or the USB host. TVS diodes sit at the connectors.\n  C101 4.7 uF (IN takes 1 to 10 uF) keeps the capacitance a USB host sees through D101 within USB's 10 uF.\n- ISET 2.0k: ICHG = KISET / RISET = 890 / 2000 = 0.445 A (KISET 797 to 975: 0.40 to 0.49 A), 0.45 C for the\n  1000 mAh pack. Precharge 88 / 2000 = 44 mA.\n- ILIM 3.3k: IIN = KILIM / RILIM = 1525 / 3300 = 0.46 A (KILIM 1330 to 1720 for 200 to 500 mA: 0.40 to 0.52 A),\n  USB 2.0 default power: the board has plain 5.1k Rd and does not read CC, and VIN-DPM is off in ILIM mode.\n  When the system load and ICHG together exceed the limit, the charger cuts ICHG (DPPM). Faster charging needs CC sensing.\n- EN2 100k to VIN_CHG, EN1 from GPIO45 with 100k to GND: (EN2, EN1) = (1, 0) selects the ILIM resistor on any input;\n  GPIO45 high gives (1, 1), USB suspend. The pull-up only draws current while input power is present\n  (EN pins have 285k internal pull-downs).\n- CE and TD to GND (charging enabled, termination on), TMR open (30 min precharge and 5 h fast-charge timers).\n- TS to the pack's 10k NTC on J101 pin 2: 75 uA bias, charging stops below about 0 to 4 C (VCOLD 2.1 V, 28k)\n  and above about 47 to 51 C (VHOT 0.30 V, 4.0k) for an NTC beta of 3950 to 3380.\n- TPS63802: VOUT = 0.5 x (1 + 560k / 100k) = 3.300 V; R2 = 100k is the datasheet maximum; MODE low (power save);\n  EN to VSYS (always on); L = 0.47 uH; 10 uF + 100 nF in, 2 x 22 uF + 100 nF out.\n  PG (open drain, 1 mA max) is TPS_PG: it pulls ESP_EN low through R212 1k (mcu_usb), so the module runs only in regulation.\n- TPS22917: CT 1 nF from CT to VIN, QOD tied to VOUT (fast discharge when the panel is switched off),\n  ON pulled down by 100k (GPIO46 strap must be low at reset).\n- MAX17048: CELL and VDD to VBAT, CTG and QSTRT to GND, ALRT only to TP107; I2C pull-ups are on the periph sheet."
 		(exclude_from_sim no)
 		(at 20.32 223.52 0)
@@
 		)
 	)
-	(global_label "ESP_EN"
+	(global_label "TPS_PG"
 		(shape bidirectional)
 		(at 88.9 180.34 0)

Commit message: fix(hardware): keep TPS63802 PG under 1 mA on the ESP32 EN network and leave the USBLC6 VBUS pin open
EN now uses R205 47k, C203 220 nF and R212 4.7k: PG sinks at most
3.3 V / 4.7k = 0.70 mA, the divider holds EN at 0.30 V or less while PG is
low, EN releases with a 10.3 ms time constant and PG glitches shorter than
about 1 ms are filtered.

U202 pin 5 is no longer tied to VBUS_USB, so the ESP32-S3's D+ pull-up
cannot back-feed the receptacle VBUS through the upper steering diode while
unplugged.

The notes boxes on both sheets state these numbers, and the mcu_usb notes
record that the U0TXD 499 ohm series resistor is inside the module.
Changed lines of the file:
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@@
 		)
 	)
-	(text_box "Values and why (datasheets: BQ24073 SLUS810N section 8.5; TPS63802 SLVSEU9D section 10; TPS22917 SLVSDW8B section 6)\n- Inputs: VBUS_USB and VBUS_DOCK each reach VIN_CHG through a PMEG2020EH Schottky (under 0.38 V at the input limit),\n  so neither input, nor a shorted dock pad, can back-feed the other or the USB host. TVS diodes sit at the connectors.\n  C101 4.7 uF (IN takes 1 to 10 uF) keeps the capacitance a USB host sees through D101 within USB's 10 uF.\n- ISET 2.0k: ICHG = KISET / RISET = 890 / 2000 = 0.445 A (KISET 797 to 975: 0.40 to 0.49 A), 0.45 C for the\n  1000 mAh pack. Precharge 88 / 2000 = 44 mA.\n- ILIM 3.3k: IIN = KILIM / RILIM = 1525 / 3300 = 0.46 A (KILIM 1330 to 1720 for 200 to 500 mA: 0.40 to 0.52 A),\n  USB 2.0 default power: the board has plain 5.1k Rd and does not read CC, and VIN-DPM is off in ILIM mode.\n  When the system load and ICHG together exceed the limit, the charger cuts ICHG (DPPM). Faster charging needs CC sensing.\n- EN2 100k to VIN_CHG, EN1 from GPIO45 with 100k to GND: (EN2, EN1) = (1, 0) selects the ILIM resistor on any input;\n  GPIO45 high gives (1, 1), USB suspend. The pull-up only draws current while input power is present\n  (EN pins have 285k internal pull-downs).\n- CE and TD to GND (charging enabled, termination on), TMR open (30 min precharge and 5 h fast-charge timers).\n- TS to the pack's 10k NTC on J101 pin 2: 75 uA bias, charging stops below about 0 to 4 C (VCOLD 2.1 V, 28k)\n  and above about 47 to 51 C (VHOT 0.30 V, 4.0k) for an NTC beta of 3950 to 3380.\n- TPS63802: VOUT = 0.5 x (1 + 560k / 100k) = 3.300 V; R2 = 100k is the datasheet maximum; MODE low (power save);\n  EN to VSYS (always on); L = 0.47 uH; 10 uF + 100 nF in, 2 x 22 uF + 100 nF out.\n  PG (open drain, 1 mA max) is TPS_PG: it pulls ESP_EN low through R212 1k (mcu_usb), so the module runs only in regulation.\n- TPS22917: CT 1 nF from CT to VIN, QOD tied to VOUT (fast discharge when the panel is switched off),\n  ON pulled down by 100k (GPIO46 strap must be low at reset).\n- MAX17048: CELL and VDD to VBAT, CTG and QSTRT to GND, ALRT only to TP107; I2C pull-ups are on the periph sheet."
+	(text_box "Values and why (datasheets: BQ24073 SLUS810N section 8.5; TPS63802 SLVSEU9D section 10; TPS22917 SLVSDW8B section 6)\n- Inputs: VBUS_USB and VBUS_DOCK each reach VIN_CHG through a PMEG2020EH Schottky (under 0.38 V at the input limit),\n  so neither input, nor a shorted dock pad, can back-feed the other or the USB host. TVS diodes sit at the connectors.\n  C101 4.7 uF (IN takes 1 to 10 uF) keeps the capacitance a USB host sees through D101 within USB's 10 uF.\n- ISET 2.0k: ICHG = KISET / RISET = 890 / 2000 = 0.445 A (KISET 797 to 975: 0.40 to 0.49 A), 0.45 C for the\n  1000 mAh pack. Precharge 88 / 2000 = 44 mA.\n- ILIM 3.3k: IIN = KILIM / RILIM = 1525 / 3300 = 0.46 A (KILIM 1330 to 1720 for 200 to 500 mA: 0.40 to 0.52 A),\n  USB 2.0 default power: the board has plain 5.1k Rd and does not read CC, and VIN-DPM is off in ILIM mode.\n  When the system load and ICHG together exceed the limit, the charger cuts ICHG (DPPM). Faster charging needs CC sensing.\n- EN2 100k to VIN_CHG, EN1 from GPIO45 with 100k to GND: (EN2, EN1) = (1, 0) selects the ILIM resistor on any input;\n  GPIO45 high gives (1, 1), USB suspend. The pull-up only draws current while input power is present\n  (EN pins have 285k internal pull-downs).\n- CE and TD to GND (charging enabled, termination on), TMR open (30 min precharge and 5 h fast-charge timers).\n- TS to the pack's 10k NTC on J101 pin 2: 75 uA bias, charging stops below about 0 to 4 C (VCOLD 2.1 V, 28k)\n  and above about 47 to 51 C (VHOT 0.30 V, 4.0k) for an NTC beta of 3950 to 3380.\n- TPS63802: VOUT = 0.5 x (1 + 560k / 100k) = 3.300 V; R2 = 100k is the datasheet maximum; MODE low (power save);\n  EN to VSYS (always on); L = 0.47 uH; 10 uF + 100 nF in, 2 x 22 uF + 100 nF out.\n  PG (open drain, sinks up to 1 mA) is TPS_PG: through R212 4.7k (mcu_usb) it sinks 0.70 mA at most and holds ESP_EN\n  at 0.30 V or less, so the module runs only in regulation (EN: 47k to +3V3, 220 nF).\n- TPS22917: CT 1 nF from CT to VIN, QOD tied to VOUT (fast discharge when the panel is switched off),\n  ON pulled down by 100k (GPIO46 strap must be low at reset).\n- MAX17048: CELL and VDD to VBAT, CTG and QSTRT to GND, ALRT only to TP107; I2C pull-ups are on the periph sheet."
 		(exclude_from_sim no)
 		(at 20.32 223.52 0)
-		(size 130.81 46.99)
+		(size 130.81 49.53)
 		(margins 1.27 1.27 1.27 1.27)
 		(stroke
