File: hardware/owl-mainboard/power.kicad_sch (KiCad schematic)
At the start: 44 parts, among them J101 Battery +, NTC, -, U101 BQ24073RGTR, U102 MAX17048G+T10, U103 TPS63802DLAR, U104 TPS22917DBVR

Commit message: fix(hardware): raise R102 to 3.6k so the charger input limit stays under 500 mA at its worst case
Parts:
- R102: value 3.3k -> 3.6k; LCSC Part # C25890 -> C25891; MPN 0402WGF3301TCE -> 0402WGF3601TCE
Changed lines of the file:
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@@
 		)
 	)
-	(text_box "Values and why (datasheets: BQ24073 SLUS810N section 8.5; TPS63802 SLVSEU9D section 10; TPS22917 SLVSDW8B section 6)\n- Inputs: VBUS_USB and VBUS_DOCK each reach VIN_CHG through a PMEG2020EH Schottky (under 0.38 V at the input limit),\n  so neither input, nor a shorted dock pad, can back-feed the other or the USB host. TVS diodes sit at the connectors.\n  C101 4.7 uF (IN takes 1 to 10 uF) keeps the capacitance a USB host sees through D101 within USB's 10 uF.\n- ISET 2.0k: ICHG = KISET / RISET = 890 / 2000 = 0.445 A (KISET 797 to 975: 0.40 to 0.49 A), 0.45 C for the\n  1000 mAh pack. Precharge 88 / 2000 = 44 mA.\n- ILIM 3.3k: IIN = KILIM / RILIM = 1525 / 3300 = 0.46 A (KILIM 1330 to 1720 for 200 to 500 mA: 0.40 to 0.52 A),\n  USB 2.0 default power: the board has plain 5.1k Rd and does not read CC, and VIN-DPM is off in ILIM mode.\n  When the system load and ICHG together exceed the limit, the charger cuts ICHG (DPPM). Faster charging needs CC sensing.\n- EN2 100k to VIN_CHG, EN1 from GPIO45 with 100k to GND: (EN2, EN1) = (1, 0) selects the ILIM resistor on any input;\n  GPIO45 high gives (1, 1), USB suspend. The pull-up only draws current while input power is present\n  (EN pins have 285k internal pull-downs).\n- CE and TD to GND (charging enabled, termination on), TMR open (30 min precharge and 5 h fast-charge timers).\n- TS to the pack's 10k NTC on J101 pin 2: 75 uA bias, charging stops below about 0 to 4 C (VCOLD 2.1 V, 28k)\n  and above about 47 to 51 C (VHOT 0.30 V, 4.0k) for an NTC beta of 3950 to 3380.\n- TPS63802: VOUT = 0.5 x (1 + 560k / 100k) = 3.300 V; R2 = 100k is the datasheet maximum; MODE low (power save);\n  EN to VSYS (always on); L = 0.47 uH; 10 uF + 100 nF in, 2 x 22 uF + 100 nF out.\n  PG (open drain, sinks up to 1 mA) is TPS_PG: through R212 4.7k (mcu_usb) it sinks 0.70 mA at most and holds ESP_EN\n  at 0.30 V or less, so the module runs only in regulation (EN: 47k to +3V3, 220 nF).\n- TPS22917: CT 1 nF from CT to VIN, QOD tied to VOUT (fast discharge when the panel is switched off),\n  ON pulled down by 100k (GPIO46 strap must be low at reset).\n- MAX17048: CELL and VDD to VBAT, CTG and QSTRT to GND, ALRT only to TP107; I2C pull-ups are on the periph sheet."
+	(text_box "Values and why (datasheets: BQ24073 SLUS810N section 8.5; TPS63802 SLVSEU9D section 10; TPS22917 SLVSDW8B section 6)\n- Inputs: VBUS_USB and VBUS_DOCK each reach VIN_CHG through a PMEG2020EH Schottky (under 0.38 V at the input limit),\n  so neither input, nor a shorted dock pad, can back-feed the other or the USB host. TVS diodes sit at the connectors.\n  C101 4.7 uF (IN takes 1 to 10 uF) keeps the capacitance a USB host sees through D101 within USB's 10 uF.\n- ISET 2.0k: ICHG = KISET / RISET = 890 / 2000 = 0.445 A (KISET 797 to 975: 0.40 to 0.49 A), 0.45 C for the\n  1000 mAh pack. Precharge 88 / 2000 = 44 mA.\n- ILIM 3.6k: IIN = KILIM / RILIM = 1525 / 3600 = 0.42 A (KILIM 1330 to 1720 for 200 to 500 mA: 0.37 to 0.48 A),\n  inside USB 2.0 default power (500 mA): the board has plain 5.1k Rd and does not read CC, and VIN-DPM is off in ILIM mode.\n  When the system load and ICHG together exceed the limit, the charger cuts ICHG (DPPM). Faster charging needs CC sensing.\n- EN2 100k to VIN_CHG, EN1 from GPIO45 with 100k to GND: (EN2, EN1) = (1, 0) selects the ILIM resistor on any input;\n  GPIO45 high gives (1, 1), USB suspend. The pull-up only draws current while input power is present\n  (EN pins have 285k internal pull-downs).\n- CE and TD to GND (charging enabled, termination on), TMR open (30 min precharge and 5 h fast-charge timers).\n- TS to the pack's 10k NTC on J101 pin 2: 75 uA bias, charging stops below about 0 to 4 C (VCOLD 2.1 V, 28k)\n  and above about 47 to 51 C (VHOT 0.30 V, 4.0k) for an NTC beta of 3950 to 3380.\n- TPS63802: VOUT = 0.5 x (1 + 560k / 100k) = 3.300 V; R2 = 100k is the datasheet maximum; MODE low (power save);\n  EN to VSYS (always on); L = 0.47 uH; 10 uF + 100 nF in, 2 x 22 uF + 100 nF out.\n  PG (open drain, sinks up to 1 mA) is TPS_PG: through R212 4.7k (mcu_usb) it sinks 0.70 mA at most and holds ESP_EN\n  at 0.30 V or less, so the module runs only in regulation (EN: 47k to +3V3, 220 nF).\n- TPS22917: CT 1 nF from CT to VIN, QOD tied to VOUT (fast discharge when the panel is switched off),\n  ON pulled down by 100k (GPIO46 strap must be low at reset).\n- MAX17048: CELL and VDD to VBAT, CTG and QSTRT to GND, ALRT only to TP107; I2C pull-ups are on the periph sheet."
 		(exclude_from_sim no)
 		(at 20.32 223.52 0)
@@
 			)
 		)
-		(property "Value" "3.3k"
+		(property "Value" "3.6k"
 			(at 111.76 118.11 0)
 			(show_name no)
@@
 			)
 		)
-		(property "LCSC Part #" "C25890"
+		(property "LCSC Part #" "C25891"
 			(at 109.22 116.84 0)
 			(hide yes)
@@
 			)
 		)
-		(property "MPN" "0402WGF3301TCE"
+		(property "MPN" "0402WGF3601TCE"
 			(at 109.22 116.84 0)
 			(hide yes)

Commit message: fix(hardware): keep the charger's paste off its open thermal vias
U101 (BQ24073 RGT) now uses a project copy of KiCad's ThermalVias
footprint, owltunes:VQFN-16-1EP_3x3mm_P0.5mm_EP1.6x1.6mm_ThermalVias_Drill0.3,
built by hw_lib_build.py: the four vias at the corners of the 1.6 mm
exposed pad are opened from 0.2 to 0.3 mm and stay open (no plugging),
and the stock paste windows, which sat over the vias, are redrawn round
them (review I2). A 1.5 x 0.6 bar and two 0.6 x 0.35 arms keep 0.1 mm
from each drill, touch no 0.5 mm via pad and print 51.6 % of the pad
(TI's guidance for RGT is roughly 50 to 80 %). The via grid moves from
0.8 to 1.1 mm pitch: at 0.8 mm no window layout clear of the vias gets
past about 31 %.

design.toml and the power sheet point U101 at the copy, and hw_sync.py
swapped it on the board in place (same position, side, rotation and
lock; KiCad saves the footprint at a new place in the file, hence the
size of the diff). hw_place.py hid U101's reference again, as Task 8
left it, and its hidden LCSC, MPN and manufacturer fields keep their
back-side orientation. The library test checks the windows against the
vias, the coverage and the copper against KiCad's footprint. DRC: no
new violation type, no lib_footprint_mismatch, parity 0.
Parts:
- U101: footprint Package_DFN_QFN:VQFN-16-1EP_3x3mm_P0.5mm_EP1.6x1.6mm -> owltunes:VQFN-16-1EP_3x3mm_P0.5mm_EP1.6x1.6mm_ThermalVias_Drill0.3
Changed lines of the file:
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@@
 			)
 		)
-		(property "Footprint" "Package_DFN_QFN:VQFN-16-1EP_3x3mm_P0.5mm_EP1.6x1.6mm"
+		(property "Footprint" "owltunes:VQFN-16-1EP_3x3mm_P0.5mm_EP1.6x1.6mm_ThermalVias_Drill0.3"
 			(at 147.32 62.23 0)
 			(hide yes)
