File: hardware/owl-mainboard/power.kicad_sch (KiCad schematic)
At the start: 45 parts, among them J101 Battery +, -, U101 BQ24073RGTR, U102 MAX17048G+T10, U103 TPS63802DLAR, U104 TPS22917DBVR

Commit message: fix(hardware): set the JLC rotation offsets the EasyEDA footprints call for
Each assembled part's EasyEDA footprint (JLC's placement zero) was matched pad by pad with
the KiCad footprint on the board. The Fabrication Toolkit writes a bottom rotation as 180
minus the KiCad rotation (the rotation seen from below, board turned over left to right,
true for all 81 bottom parts) plus its own table rotation, so a part needs the
EasyEDA-to-KiCad angle less the table's angle. Five parts get an FT Rotation Offset:

- D101, D102 (PMEG2020EH, C456104): 180. EasyEDA's footprint has pad 1, the cathode, on
  the right at zero; KiCad's D_SOD-123F has it on the left. No toolkit rule. CPL 180 -> 0.
- J101 (S2B-PH-SM4-TB, C295747): 180. EasyEDA's footprint matches KiCad's at zero; the
  toolkit's ^JST_PH_S rule adds 180, which this cancels. CPL 270 -> 90.
- U202 (USBLC6-2SC6, C7519): 90. EasyEDA's SOT-23-6 BL footprint (pin 1 bottom left, rows
  horizontal) is 270 from KiCad's; the toolkit's ^SOT-23 rule gives 180. CPL 180 -> 270.
- U303 (LIS2DW12TR, C189624): 270. EasyEDA's LGA-12 BL footprint runs pins 1 to 4 along
  the bottom, KiCad's down the left (ruling R30); no toolkit rule. CPL 180 -> 90.

The offsets live in design.toml (rotation_offset) and on the symbols; hw_sync.py now copies
the field to the footprint, where the toolkit reads it, hw_bom.py checks symbol against
design.toml and a test checks footprint against design.toml. JLC's placement preview
confirms them at order time. ordering.md and the review record the offsets and the method.

ERC 0, DRC 0/0/0 with parity, hw_fab 0 errors (top 6, bottom 81), Gerbers unchanged.
Parts:
- D101, D102, J101: FT Rotation Offset (none) -> 180
Changed lines of the file:
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@@
+			)
+		)
+		(property "FT Rotation Offset" "180"
+			(at 40.64 66.04 0)
+			(hide yes)
+			(show_name no)
+			(do_not_autoplace no)
+			(effects
+				(font
+					(size 1.27 1.27)
+				)
 			)
 		)
@@
 			)
 		)
+		(property "FT Rotation Offset" "180"
+			(at 198.12 76.2 0)
+			(hide yes)
+			(show_name no)
+			(do_not_autoplace no)
+			(effects
+				(font
+					(size 1.27 1.27)
+				)
+			)
+		)
 		(pin "1"
 		)
@@
 			(at 40.64 50.8 0)
 			(hide yes)
+			(show_name no)
+			(do_not_autoplace no)
+			(effects
+				(font
+					(size 1.27 1.27)
+				)
+			)
+		)
+		(property "FT Rotation Offset" "180"
+			(at 40.64 50.8 0)
+			(hide yes)

Commit message: fix(hardware): set the charge current to at most 0.5 C of the 700 mAh pack
Controller ruling: the BQ24073 fast-charge current may not exceed 0.5 C of the EEMB 700 mAh
fallback pack, 0.35 A. ICHG = KISET / RISET with KISET 797, 890, 975 A-ohm (SLUS810N p. 13);
with KISET at 975 and the resistor 1 % low, RISET must be at least 975 / 0.35 / 0.99 = 2.81k.
JLC lists 2.8k (C62741), 2.87k (C113479), 2.94k (C25886) and 3k (C25784) as Extended; the
nearest Basic value at or above is 3.3k, 0402WGF3301TCE (C25890, 1986011 in stock).

R101 2k (C4109) -> 3.3k (C25890): ICHG 0.270 A typical, 0.239 to 0.298 A (0.43 C of 700 mAh,
0.40 C of 740 mAh at worst); precharge 27 mA, termination about 27 mA. ICHG is now below the
input limit (0.369 to 0.478 A), so the cell charges at ICHG unless the system load takes the
input to its limit. U101's worst-case dissipation falls from about 0.77 W to 0.51 W.

design.toml, the schematic value and fields, the board (hw_sync), rev-a.md (calculations, the
smaller-cell note, the RT101 bring-up item, a decisions row), bringup.md step 9 and the review's
BQ24073 and thermal rows follow. hw_fab 0 errors (top 6, bottom 81; BOM row R101 3.3k C25890),
hw_stock 43 unique parts, 0 low; ERC 0, DRC 0/0/0 with parity, check_all 0, tools tests 110.
Parts:
- R101: value 2k -> 3.3k; LCSC Part # C4109 -> C25890; MPN 0402WGF2001TCE -> 0402WGF3301TCE
Changed lines of the file:
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@@
 			)
 		)
-		(property "Value" "2k"
+		(property "Value" "3.3k"
 			(at 101.6 118.11 0)
 			(show_name no)
@@
 			)
 		)
-		(property "LCSC Part #" "C4109"
+		(property "LCSC Part #" "C25890"
 			(at 99.06 116.84 0)
 			(hide yes)
@@
 			)
 		)
-		(property "MPN" "0402WGF2001TCE"
+		(property "MPN" "0402WGF3301TCE"
 			(at 99.06 116.84 0)
 			(hide yes)
