File: hardware/owl-mainboard/mcu_usb.kicad_sch (KiCad schematic)
At the start: 34 parts, among them J201 USB-C, J202 EXP: GND, 3V3, A, B, SW201 Ear left, SW202 Ear right, SW203 Beak, U201 ESP32-S3-WROOM-1-N16R8, U202 USBLC6-2SC6, Y201 32.768kHz 12.5pF

Commit message: fix(hardware): move the CPL points of U201, J201 and the perch J1 to JLC's origins
The Fabrication Toolkit puts an SMD part's CPL point on the KiCad footprint's anchor; JLC places
its EasyEDA footprint by that footprint's origin. Fitting every assembled part's EasyEDA
footprint onto the board pads by pad number puts the two within 0.075 mm for all parts but
three, where the KiCad anchor is the body centre and EasyEDA's origin is near the pad pattern's
centre:

- U201 (ESP32-S3-WROOM-1, C2913202), bottom, KiCad rotation 180: EasyEDA origin at owl
  (0, 26.723), anchor (0, 30.35). The toolkit turns a bottom offset (x, y) at 180 into (-x, y),
  so FT Position Offset "0,-3.627". CPL (0, 30.35) -> (0, 26.723).
- J201 (TYPE-C-31-M-12, C165948), bottom, rotation 180: origin (-12, -32.229), anchor
  (-12, -33.8): "0,1.571". CPL (-12, -33.8) -> (-12, -32.229).
- Perch J1 (same receptacle), top, rotation 90: the toolkit turns (x, y) into (-y, x); origin
  (12.229, -1.5), anchor (13.8, -1.5): "0,1.571". CPL (13.8, -1.5) -> (12.229, -1.5).

Stored like the rotation offsets: design.toml position_offset, the symbol field, and the
footprint field through hw_sync.py (FIELDS gains "FT Position Offset"); hw_bom.py checks symbol
against design.toml and the sync test checks footprints against design.toml on both boards.
The review and ordering.md say the preview checks these three positions as well as rotations.

hw_fab 0 errors on both boards (main top 6, bottom 81; perch top 15), ERC 0, DRC 0/0/0 with
parity on both, check_all 0, tools tests 110 passed.
Parts:
- J201: FT Position Offset (none) -> 0,1.571
- U201: FT Position Offset (none) -> 0,-3.627
Changed lines of the file:
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@@
 			)
 		)
+		(property "FT Position Offset" "0,-3.627"
+			(at 228.6 132.08 0)
+			(hide yes)
+			(show_name no)
+			(do_not_autoplace no)
+			(effects
+				(font
+					(size 1.27 1.27)
+				)
+			)
+		)
 		(pin "1"
 		)
@@
 			(at 35.56 71.12 0)
 			(hide yes)
+			(show_name no)
+			(do_not_autoplace no)
+			(effects
+				(font
+					(size 1.27 1.27)
+				)
+			)
+		)
+		(property "FT Position Offset" "0,1.571"
+			(at 35.56 71.12 0)
+			(hide yes)
